Commit message: it exists and walks now

File: src/rm_description/urdf/gazebo_control.xacro (robot description, xacro)
@@ -5,8 +5,8 @@
         <plugin name="gz::sim::systems::DiffDrive" filename="gz-sim-diff-drive-system">
             <!-- Juntas das rodas (devem corresponder ao differetial_robot.xacro) -->
-            <left_joint>left_wheel_joint</left_joint>
-            <right_joint>right_wheel_joint</right_joint>
-            <wheel_separation>0.35</wheel_separation>
-            <wheel_radius>0.05</wheel_radius>
+            <left_joint>caixa_rodaL</left_joint>
+            <right_joint>caixa_rodaR</right_joint>
+            <wheel_separation>.62</wheel_separation>
+            <wheel_radius>0.15</wheel_radius>
             <!-- Limites -->
             <max_wheel_torque>200</max_wheel_torque>
@@ -26,6 +26,6 @@
             name="gz::sim::systems::JointStatePublisher">
             <topic>joint_states</topic>
-            <joint_name>left_wheel_joint</joint_name>
-            <joint_name>right_wheel_joint</joint_name>
+            <joint_name>caixa_rodaL</joint_name>
+            <joint_name>caixa_rodaR</joint_name>
         </plugin>
     </gazebo>

File: src/rm_description/urdf/macros.xacro (robot description, xacro)
@@ -46,5 +46,4 @@
         <origin xyz="0 0 0" rpy="0 0 0"/>
         <mass value="${mass}"/>
-        <!-- Fórmula de inércia para esfera sólida -->
         <inertia
           ixx="${(2/5) * mass * radius * radius}"

File: src/rm_description/urdf/properties.xacro (robot description, xacro)
@@ -22,5 +22,8 @@
   <!-- ============================================ -->
   <material name="gray">
-    <color rgba="0.5 0.5 0.5 1"/>
+    <color rgba="0.412 0.412 0.412 1"/>
+  </material>
+  <material name="pink">
+    <color rgba="1 0.412 0.706 1"/>
   </material>
 </robot>

File: src/rm_description/urdf/robot.xacro (robot description, xacro)
@@ -14,4 +14,5 @@
   <xacro:include filename="$(find rm_description)/urdf/properties.xacro"/>
   <xacro:include filename="$(find rm_description)/urdf/macros.xacro"/>
+  <xacro:include filename="$(find rm_description)/urdf/gazebo_control.xacro" />
   <!-- ==================== -->
   <!-- BASE FOOTPRINT       -->
@@ -22,10 +23,10 @@
   <visual>
     <origin xyz="0 0 0" rpy="0 0 0"/>
-    <geometry> <box size=".5 1 0.1"/> </geometry>
-    <material name="gray"/>
+    <geometry> <box size=".5 .5 0.1"/> </geometry>
+    <material name="pink"/>
   </visual>
   <collision>
     <origin xyz="0 0 0" rpy="0 0 0"/>
-    <geometry> <box size=".5 1 0.1"/> </geometry>
+    <geometry> <box size=".5 .5 0.1"/> </geometry>
   </collision>
   <inertial>
@@ -38,5 +39,5 @@
     <parent link="base_footprint"/>
     <child link="caixa"/>
-    <origin xyz="0 0 0.025" rpy="0 0 0"/>
+    <origin xyz="0 0 ${0.025+.15}" rpy="0 0 0"/>
   </joint>
   <xacro:cylinder_link
@@ -49,6 +50,6 @@
     <parent link="caixa"/>
     <child link="rodaL"/>
-    <origin xyz="0 ${(1/2)+.05} 0" rpy="300 0 0"/>
-    <axis xyz="0 0 1"/>
+    <origin xyz="0 ${(1/4)+.01+.1} 0" rpy="${pi/2} 0 0"/>
+    <axis xyz="0 0 -1"/>
   </joint>
   <xacro:cylinder_link
@@ -61,6 +62,6 @@
     <parent link="caixa"/>
     <child link="rodaR"/>
-    <origin xyz="0 -${(1/2)+.05} 0" rpy="300 0 0"/>
-    <axis xyz="0 0 1"/>
+    <origin xyz="0 -${(1/4)+.01} 0" rpy="${pi/2} 0 0"/>
+    <axis xyz="0 0 -1"/>
   </joint>
   <xacro:sphere_link
@@ -68,5 +69,5 @@
     radius="${.15}"
     mass="${1.0}"
-    material="gray"/>
+    material="pink"/>
   <joint name="caixa_head" type="fixed">
     <parent link="caixa"/>
