Commit message: supostamente aps1

File: src/rm_description/urdf/robot.urdf.xacro (robot description, xacro)
@@ -3,3 +3,4 @@
     <xacro:include filename="$(find rm_description)/urdf/robot.xacro" />
     <xacro:include filename="$(find rm_description)/urdf/gazebo_control.xacro" />
+    <xacro:include filename="$(find rm_description)/urdf/sensors.xacro" />
 </robot>

File: src/rm_description/urdf/robot.xacro (robot description, xacro)
@@ -67,5 +67,5 @@
   <xacro:sphere_link
     name="head"
-    radius="${.15}"
+    radius="${.075}"
     mass="${1.0}"
     material="pink"/>
@@ -73,5 +73,29 @@
     <parent link="caixa"/>
     <child link="head"/>
-    <origin xyz=".25 0 0" rpy="0 0 0"/>
+    <origin xyz=".25 0 -0.075" rpy="0 0 0"/>
   </joint>
+  <xacro:cylinder_link
+    name="camera"
+    length="${.1}"
+    radius="${.05}"
+    mass="${1.0}"
+    material="pink"/>
+  <joint name="caixa_camera" type="fixed">
+    <parent link="caixa"/>
+    <child link="camera"/>
+    <origin xyz="0.05 0 .01" rpy="0 0 0"/>
+  </joint>
+  <xacro:cylinder_link
+    name="lidar"
+    length="${.15+.01}"
+    radius="${.05}"
+    mass="${1.0}"
+    material="pink"/>
+  <joint name="caixa_lidar" type="fixed">
+    <parent link="caixa"/>
+    <child link="lidar"/>
+    <origin xyz="0 0 .01" rpy="0 0 0"/>
+  </joint>
+  <link name="imu">
+  </link>
 </robot>
